Commit message: add common model for franka_arm and separate pedestal

File: robots/panda/models/panda.urdf.xacro (robot description, xacro)
@@ -1,5 +1,8 @@
 <?xml version="1.0"?>
 <robot xmlns:xacro="http://www.ros.org/wiki/xacro" name="panda" >
+  <!-- arguments -->
+  <xacro:arg name="arm_id" default="panda" />
   <xacro:arg name="hand" default="true" /> <!-- enable defalut hand -->
-  <xacro:include filename="$(find franka_description)/robots/panda/panda.urdf.xacro" />
+  <!-- load -->
+  <xacro:include filename="$(find panda)/models/franka_arm.urdf.xacro" />
 </robot>

File: robots/panda/models/panda_pedestal.urdf.xacro (robot description, xacro)
@@ -1,52 +1,8 @@
 <?xml version="1.0"?>
 <robot xmlns:xacro="http://www.ros.org/wiki/xacro" name="panda_pedestal" >
+  <!-- arguments -->
+  <xacro:arg name="arm_id" default="panda" />
   <xacro:arg name="hand" default="true" /> <!-- enable defalut hand -->
-  <xacro:include filename="$(find franka_description)/robots/panda/panda.urdf.xacro" />
-  <!-- base -->
-  <link name="world" />
-  <joint name="world_to_panda" type="fixed">
-    <origin xyz="0 0 0.79" rpy="0 0 0"/>  <!-- Pedestal height [mm] from its drawing. 800 (stand leg), 790 (wheel) -->
-    <parent link="world"/>
-    <child link="panda_link0"/>
-  </joint>
-  <!-- pedestal -->
-  <xacro:property name="arm_to_pedestal_x" value="-0.0445" />  <!-- Based on pedestal's CAD and panda's footprint (https://www.generationrobots.com/media/panda-franka-emika-datasheet.pdf) -->
-  <xacro:macro name="pedestal" params="arm_id">
-    <link name="${arm_id}_pedestal">
-      <visual>
-        <origin xyz="0.0 0.0 0.0" rpy="0.0 0.0 0.0" />
-        <geometry>
-          <mesh filename="package://panda_eus/meshes/pedestal.stl" scale="0.001 0.001 0.001" />
-        </geometry>
-        <material name="metal">
-          <color rgba="0.75 0.75 0.75 1.0" />
-        </material>
-      </visual>
-      <collision>
-        <origin xyz="0.0 0.0 -0.252" rpy="0.0 0.0 0.0" />
-        <geometry>
-          <cylinder radius="0.115" length="0.504" />
-        </geometry>
-      </collision>
-      <collision>
-        <origin xyz="0.10675 0.0 -0.652" rpy="0.0 0.0 0.0" />
-        <geometry>
-          <box size="0.7135 0.68 0.296" />
-        </geometry>
-      </collision>
-    </link>
-    <joint name="${arm_id}_pedestal_joint" type="fixed">
-      <parent link="${arm_id}_link0" />
-      <child  link="${arm_id}_pedestal" />
-      <origin xyz="${arm_to_pedestal_x} 0.0 0.0" rpy="0.0 0.0 0.0" />
-    </joint>
-    <inertial>
-      <!-- We do not know true inertial parameters -->
-      <mass value="1000" />
-      <origin rpy="0 0 0" xyz="0.0 0.0 -0.4" />
-      <inertia ixx="10.0" ixy="0.0" ixz="0.0"
-               iyy="10.0" iyz="0.0" izz="10.0" />
-    </inertial>
-  </xacro:macro>
-  <xacro:pedestal arm_id="panda" />
+  <!-- load -->
+  <xacro:include filename="$(find panda)/models/franka_arm_pedestal.urdf.xacro" />
 </robot>
