Commit message: change magician_description to dobot_magician_description

File: robots/dobot_magician/dobot_magician_description/urdf/demo.urdf (robot description, URDF)
Before this commit: robot magician, 6 links, 5 joints
Links:
- link base_link: geometry collision mesh filename=package://dobot_magician_description/meshes/base_link.STL; visual mesh filename=package://dobot_magician_description/meshes/base_link.STL
- link link_1: geometry collision mesh filename=package://dobot_magician_description/meshes/link_1.STL; visual mesh filename=package://dobot_magician_description/meshes/link_1.dae
- link link_2: geometry collision mesh filename=package://dobot_magician_description/meshes/link_2.STL; visual mesh filename=package://dobot_magician_description/meshes/link_2.dae
- link link_5: geometry collision mesh filename=package://dobot_magician_description/meshes/link_5.dae; visual mesh filename=package://dobot_magician_description/meshes/link_5.dae
- link link_6: geometry collision mesh filename=package://dobot_magician_description/meshes/link_6.STL; visual mesh filename=package://dobot_magician_description/meshes/link_6.STL
- link link_7: geometry collision mesh filename=package://dobot_magician_description/meshes/link_7.STL; visual mesh filename=package://dobot_magician_description/meshes/link_7.STL

File: robots/dobot_magician/dobot_magician_moveit_config/config/gazebo_magician.urdf (robot description, URDF)
Before this commit: robot magician, 6 links, 5 joints
Links:
- link base_link: geometry collision mesh filename=package://dobot_magician_description/meshes/base_link.STL; visual mesh filename=package://dobot_magician_description/meshes/base_link.STL
- link link_1: geometry collision mesh filename=package://dobot_magician_description/meshes/link_1.STL; visual mesh filename=package://dobot_magician_description/meshes/link_1.dae
- link link_2: geometry collision mesh filename=package://dobot_magician_description/meshes/link_2.STL; visual mesh filename=package://dobot_magician_description/meshes/link_2.dae
- link link_5: geometry collision mesh filename=package://dobot_magician_description/meshes/link_5.dae; visual mesh filename=package://dobot_magician_description/meshes/link_5.dae
- link link_6: geometry collision mesh filename=package://dobot_magician_description/meshes/link_6.STL; visual mesh filename=package://dobot_magician_description/meshes/link_6.STL
- link link_7: geometry collision mesh filename=package://dobot_magician_description/meshes/link_7.STL; visual mesh filename=package://dobot_magician_description/meshes/link_7.STL
