Commit message: modify pedastal description for displaying multiple franka_arm at once

File: robots/franka_arm/models/fr3_pedestal.urdf.xacro (robot description, xacro)
@@ -1,8 +1,11 @@
 <?xml version="1.0"?>
 <robot xmlns:xacro="http://www.ros.org/wiki/xacro" name="fr3_pedestal" >
-  <!-- arguments -->
-  <xacro:arg name="arm_id" default="fr3" />
-  <xacro:arg name="hand" default="true" /> <!-- enable defalut hand -->
-  <!-- load -->
+  <!-- paremeters -->
+  <xacro:arg name="franka_arm_pedestal_id"     default="fr3" />
+  <xacro:arg name="franka_arm_pedestal_origin" default="world" />
+  <xacro:arg name="franka_arm_pedestal_hand"   default="true" />
+  <xacro:property name="franka_arm_pedestal_joint_limits" default="${xacro.load_yaml('$(find franka_description)/robots/$(arg franka_arm_pedestal_id)/joint_limits.yaml')}" />
+  <!-- franka_arm_pedestal -->
   <xacro:include filename="$(find franka_arm)/models/franka_arm_pedestal.urdf.xacro" />
+  <xacro:franka_arm_pedestal franka_arm_pedestal_id="$(arg franka_arm_pedestal_id)" franka_arm_pedestal_origin="$(arg franka_arm_pedestal_origin)" franka_arm_pedestal_joint_limits="${franka_arm_pedestal_joint_limits}" franka_arm_pedestal_hand="$(arg franka_arm_pedestal_hand)" />
 </robot>

File: robots/franka_arm/models/franka_arm_pedestal.urdf.xacro (robot description, xacro)
@@ -1,26 +1,21 @@
 <?xml version="1.0"?>
 <robot xmlns:xacro="http://www.ros.org/wiki/xacro" name="franka_arm_pedestal" >
-  <!-- arguments -->
-  <xacro:arg name="arm_id" default="panda" />
-  <xacro:arg name="arm_origin" default="world" />
-  <!-- load -->
-  <xacro:include filename="$(find franka_description)/robots/$(arg arm_id)/$(arg arm_id).urdf.xacro" />
-  <xacro:include filename="$(find franka_arm)/models/pedestal.urdf.xacro" />
+  <!-- paremeters -->
+  <xacro:property name="franka_arm_pedestal_origin_xyz" value="0 0 0.79" />  <!-- Pedestal height [mm] from its drawing. 800 (stand leg), 790 (wheel) -->
   <!-- macro -->
-  <xacro:macro name="franka_arm_pedastal"
-               params="arm_id
-                       arm_origin:='world'
-                       ">
-    <!-- generate the link where the robot attached to-->
-    <link name="${arm_origin}" />
-    <joint name="${arm_origin}_to_$(arg arm_id)" type="fixed">
-      <origin xyz="0 0 0.79" rpy="0 0 0"/>  <!-- Pedestal height [mm] from its drawing. 800 (stand leg), 790 (wheel) -->
-      <parent link="${arm_origin}"/>
-      <child  link="$(arg arm_id)_link0"/>
-    </joint>
+  <xacro:macro name="franka_arm_pedestal" params="franka_arm_pedestal_id:='panda' franka_arm_pedestal_origin:='world' franka_arm_pedestal_joint_limits:='' franka_arm_pedestal_hand:='true'" >
+    <!-- arm -->
+    <xacro:include filename="$(find franka_description)/robots/common/franka_arm.xacro" />
+    <xacro:franka_arm arm_id="${franka_arm_pedestal_id}" connected_to="${franka_arm_pedestal_origin}" xyz="${franka_arm_pedestal_origin_xyz}" safety_distance="0.03" joint_limits="${franka_arm_pedestal_joint_limits}"/>
+    <!-- hand -->
+    <xacro:if value="${franka_arm_pedestal_hand}">
+      <xacro:include filename="$(find franka_description)/robots/common/franka_hand.xacro" />
+      <xacro:franka_hand arm_id="${franka_arm_pedestal_id}" rpy="0 0 ${-pi/4}" connected_to="${franka_arm_pedestal_id}_link8" safety_distance="0.03"/>
+    </xacro:if>
+    <!-- generate the link where the robot connected to-->
+    <link name="${franka_arm_pedestal_origin}" />
+    <!-- pedestal -->
+    <xacro:include filename="$(find franka_arm)/models/pedestal.urdf.xacro" />
+    <xacro:pedestal arm_id="${franka_arm_pedestal_id}" />
   </xacro:macro>
-  <!-- franka_arm_pedastal -->
-  <xacro:franka_arm_pedastal arm_id="$(arg arm_id)" arm_origin="$(arg arm_origin)" />
-  <!-- pedestal -->
-  <xacro:pedestal arm_id="$(arg arm_id)" />
 </robot>

File: robots/franka_arm/models/panda_pedestal.urdf.xacro (robot description, xacro)
@@ -1,8 +1,11 @@
 <?xml version="1.0"?>
 <robot xmlns:xacro="http://www.ros.org/wiki/xacro" name="panda_pedestal" >
-  <!-- arguments -->
-  <xacro:arg name="arm_id" default="panda" />
-  <xacro:arg name="hand" default="true" /> <!-- enable defalut hand -->
-  <!-- load -->
+  <!-- paremeters -->
+  <xacro:arg name="franka_arm_pedestal_id"     default="panda" />
+  <xacro:arg name="franka_arm_pedestal_origin" default="world" />
+  <xacro:arg name="franka_arm_pedestal_hand"   default="true" />
+  <xacro:property name="franka_arm_pedestal_joint_limits" default="${xacro.load_yaml('$(find franka_description)/robots/$(arg franka_arm_pedestal_id)/joint_limits.yaml')}" />
+  <!-- franka_arm_pedestal -->
   <xacro:include filename="$(find franka_arm)/models/franka_arm_pedestal.urdf.xacro" />
+  <xacro:franka_arm_pedestal franka_arm_pedestal_id="$(arg franka_arm_pedestal_id)" franka_arm_pedestal_origin="$(arg franka_arm_pedestal_origin)" franka_arm_pedestal_joint_limits="${franka_arm_pedestal_joint_limits}" franka_arm_pedestal_hand="$(arg franka_arm_pedestal_hand)"/>
 </robot>
